File: FPGABoardKiCad/FPGABOARD/FPGABOARD.kicad_sch (KiCad schematic)
At the start: 80 parts, among them J1 USB_C_Receptacle_USB2.0_14P, J2 Program, J3 12PMOD, J4 6PMOD, J6 Conn_02x13_Odd_Even, SW1 ResetICE, SW2 BTN0, SW3 BTN1, SW4 BTN2, U1 AP2127K-1.2, U2 AP2127K-3.3, U3 W25Q32JVSS, U4 93LCxxBxxOT, U5 FT2232HPQ, U6 IS62LV256AL, U7 ICE40HX1K-VQ100, Y1 SG-210STF, Y2 SG-210STF

Commit message: schematic image
Parts:
- C14, C15, C16, C17, C18, C19, C20, C21, C22, C24, C25, C26, C27, C28, C29, C30, C31, C32, C34: footprint Capacitor_SMD:C_0603_1608Metric -> Capacitor_SMD:C_0603_1608Metric_Pad1.08x0.95mm_HandSolder
- R9: footprint Resistor_SMD:R_0603_1608Metric -> Resistor_SMD:R_0603_1608Metric_Pad0.98x0.95mm_HandSolder
Other:
- note added: "CLOCKs"
- note added: "FT2232"
- note added: "ICE40 FPGA"
- note added: "LED & BUTTONS"
- note added: "MEMORY"
- note added: "PIN HEADERS"
- note added: "POWER"
- note added: "RAM"
- note added: "STATUS & RESET"
- moved on the sheet: C1, C10, C2, C22, C24, C25, C26, C27, C28, C29, C30, C31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
