File: FPGABoardKiCad/FPGABOARD/FPGABOARD.kicad_pcb (KiCad board)
At the start: 4 copper layers, 78 x 51 mm, 80 parts, among them J1 USB_C_Receptacle_USB2.0_14P, J2 Program, J3 12PMOD, J4 6PMOD, J6 Conn_02x13_Odd_Even, SW1 ResetICE, SW2 BTN0, SW3 BTN1, SW4 BTN2, U1 AP2127K-1.2, U2 AP2127K-3.3, U3 W25Q32JVSS, U4 93LCxxBxxOT, U5 FT2232HPQ, U6 IS62LV256AL, U7 ICE40HX1K-VQ100, Y1 SG-210STF, Y2 SG-210STF

Commit message: schematic image
Parts:
- C14, C15, C16, C17, C18, C19, C20, C21, C22, C24, C25, C26, C27, C28, C29, C30, C31, C32, C34: footprint Capacitor_SMD:C_0603_1608Metric -> Capacitor_SMD:C_0603_1608Metric_Pad1.08x0.95mm_HandSolder
- R9: footprint Resistor_SMD:R_0603_1608Metric -> Resistor_SMD:R_0603_1608Metric_Pad0.98x0.95mm_HandSolder
Routing:
- net +1V2: track 35.8 -> 36.6 mm
- net GND: track 124.2 -> 124.9 mm
- net /EXP7: track 31.4 -> 31.9 mm, vias 0 -> 2
Other:
- board text added: "3V3"
- board text added: "5V"
- board text added: "CDN"
- board text added: "DYNIX7"
- board text added: "GND"
- board text added: "Johnny Chen"
- board text added: "RST"
- board text added: "SCK"
- board text added: "SCL"
- board text added: "SDA"
- board text added: "SDI"
- board text added: "SDO"
- board text added: "SS"
